Commit message: Add gazebo properties and sensors

File: spot_description/urdf/spot.urdf (robot description, URDF)
Before this commit: robot spot, 18 links, 17 joints
Links:
- link base: geometry collision box size=0.7 0.3 0.2; visual mesh filename=file:///home/kuba/fun/ros/spot/src/spot/spot_description/me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
- link fl_hip: geometry visual mesh filename=file:///home/kuba/fun/ros/spot/src/spot/spot_description/me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
- link fl_lleg: geometry collision sphere radius=0.035; visual mesh filename=file:///home/kuba/fun/ros/spot/src/spot/spot_description/me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
- link fl_uleg: geometry visual mesh filename=file:///home/kuba/fun/ros/spot/src/spot/spot_description/me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
- link fr_hip: geometry visual mesh filename=file:///home/kuba/fun/ros/spot/src/spot/spot_description/me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
- link fr_lleg: geometry collision sphere radius=0.035; visual mesh filename=file:///home/kuba/fun/ros/spot/src/spot/spot_description/me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
- link fr_uleg: geometry visual mesh filename=file:///home/kuba/fun/ros/spot/src/spot/spot_description/me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
- link hl_hip: geometry visual mesh filename=file:///home/kuba/fun/ros/spot/src/spot/spot_description/me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
- link hl_lleg: geometry collision sphere radius=0.035; visual mesh filename=file:///home/kuba/fun/ros/spot/src/spot/spot_description/me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
- link hl_uleg: geometry visual mesh filename=file:///home/kuba/fun/ros/spot/src/spot/spot_description/me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
- link hr_hip: geometry visual mesh filename=file:///home/kuba/fun/ros/spot/src/spot/spot_description/me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
- link hr_lleg: geometry collision sphere radius=0.035; visual mesh filename=file:///home/kuba/fun/ros/spot/src/spot/spot_description/me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
- link hr_uleg: geometry visual mesh filename=file:///home/kuba/fun/ros/spot/src/spot/spot_description/me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
